File: Placa central/Placa_central_v01/Placa_central_v01.sch (KiCad schematic (older format))
At the start: 21 parts

Commit message: Aprimorado trabalho ja feito
Separando os arquivos da maneira correta, criando a biblioteca, associando componentes certos, acertando questão de variáveis de PATH e etc.
Tentativa de criar uma metodologia para as libraries e outros documentos do projeto.
Parts:
- C1, C2: renamed from C?; footprint (none) -> Capacitors_THT:CP_Axial_L11.0mm_D5.0mm_P18.00mm_Horizontal
- D1, D2, D3: renamed from D?; footprint (none) -> Capacitors_THT:CP_Axial_L11.0mm_D5.0mm_P18.00mm_Horizontal
- Q1: renamed from Q?; footprint (none) -> Capacitors_THT:CP_Axial_L11.0mm_D5.0mm_P18.00mm_Horizontal
- Q2, Q3: renamed from Q?; footprint (none) -> Sensores_e_componentes_SL:TCRT5000
- U1, U2: renamed from U?; symbol cyclophone:TCRT5000 -> Placa_central_v01-rescue:TCRT5000-cyclophone
- gave numbers to parts that had none: 11
Changed lines of the file:
@@
 EESchema Schematic File Version 4
+LIBS:Placa_central_v01-cache
 EELAYER 26 0
 EELAYER END
@@
 $EndDescr
 $Comp
-L MCU_Module:Arduino_Nano_v3.x A?
+L MCU_Module:Arduino_Nano_v3.x A1
 U 1 1 5C812F31
 P 3250 2750
-F 0 "A?" H 3250 1664 50  0000 C CNN
+F 0 "A1" H 3250 1664 50  0000 C CNN
 F 1 "Arduino_Nano_v3.x" H 3250 1573 50  0000 C CNN
 F 2 "Module:Arduino_Nano" H 3400 1800 50  0001 L CNN
@@
 $EndComp
 $Comp
-L cyclophone:TCRT5000 U?
+L Placa_central_v01-rescue:TCRT5000-cyclophone U2
 U 1 1 5C812FD5
 P 9450 2400
-F 0 "U?" H 9450 2550 60  0000 C CNN
+F 0 "U2" H 9450 2550 60  0000 C CNN
 F 1 "TCRT5000" H 9450 2650 60  0000 C CNN
-F 2 "" H 9450 2400 60  0000 C CNN
+F 2 "" H 9450 2400 60  0001 C CNN
 F 3 "" H 9450 2400 60  0000 C CNN
 	1    9450 2400
@@
 $EndComp
 $Comp
-L Device:R R?
+L Device:R R5
 U 1 1 5C8132E2
 P 10150 2450
-F 0 "R?" V 9943 2450 50  0000 C CNN
+F 0 "R5" V 9943 2450 50  0000 C CNN
 F 1 "330" V 10034 2450 50  0000 C CNN
 F 2 "" V 10080 2450 50  0001 C CNN
@@
 $EndComp
 $Comp
-L Device:R R?
+L Device:R R6
 U 1 1 5C813322
 P 10150 2700
-F 0 "R?" V 9943 2700 50  0000 C CNN
+F 0 "R6" V 9943 2700 50  0000 C CNN
 F 1 "11k" V 10034 2700 50  0000 C CNN
 F 2 "" V 10080 2700 50  0001 C CNN
@@
 	9950 2700 10000 2700
 $Comp
-L cyclophone:TCRT5000 U?
+L Placa_central_v01-rescue:TCRT5000-cyclophone U1
 U 1 1 5C8139FF
 P 9450 1450
-F 0 "U?" H 9450 1600 60  0000 C CNN
+F 0 "U1" H 9450 1600 60  0000 C CNN
 F 1 "TCRT5000" H 9450 1700 60  0000 C CNN
-F 2 "" H 9450 1450 60  0000 C CNN
+F 2 "" H 9450 1450 60  0001 C CNN
 F 3 "" H 9450 1450 60  0000 C CNN
 	1    9450 1450
@@
 $EndComp
 $Comp
-L Device:R R?
+L Device:R R3
 U 1 1 5C813A06
 P 10150 1500
-F 0 "R?" V 9943 1500 50  0000 C CNN
+F 0 "R3" V 9943 1500 50  0000 C CNN
 F 1 "330" V 10034 1500 50  0000 C CNN
 F 2 "" V 10080 1500 50  0001 C CNN
@@
 $EndComp
 $Comp
-L Device:R R?
+L Device:R R4
 U 1 1 5C813A0D
 P 10150 1750
-F 0 "R?" V 9943 1750 50  0000 C CNN
+F 0 "R4" V 9943 1750 50  0000 C CNN
 F 1 "11k" V 10034 1750 50  0000 C CNN
 F 2 "" V 10080 1750 50  0001 C CNN
@@
 Encoder2
 $Comp
-L Regulator_Linear:L7805 U?
+L Regulator_Linear:L7805 U3
 U 1 1 5C81568D
 P 9600 3550
-F 0 "U?" H 9600 3792 50  0000 C CNN
+F 0 "U3" H 9600 3792 50  0000 C CNN
 F 1 "L7805" H 9600 3701 50  0000 C CNN
 F 2 "" H 9625 3400 50  0001 L CIN
@@
 GND
 $Comp
-L cyclophone:C C?
+L cyclophone:C C1
 U 1 1 5C81583B
 P 9150 3750
-F 0 "C?" H 9265 3788 40  0000 L CNN
+F 0 "C1" H 9265 3788 40  0000 L CNN
 F 1 "0.33uF" H 9265 3712 40  0000 L CNN
-F 2 "" H 9188 3600 30  0000 C CNN
+F 2 "Capacitors_THT:CP_Axial_L11.0mm_D5.0mm_P18.00mm_Horizontal" H 9188 3600 30  0001 C CNN
 F 3 "" H 9150 3750 60  0000 C CNN
 	1    9150 3750
@@
 $EndComp
 $Comp
-L cyclophone:C C?
+L cyclophone:C C2
 U 1 1 5C8158B3
 P 10050 3750
-F 0 "C?" H 10165 3788 40  0000 L CNN
+F 0 "C2" H 10165 3788 40  0000 L CNN
 F 1 "0.1uF" H 10165 3712 40  0000 L CNN
-F 2 "" H 10088 3600 30  0000 C CNN
+F 2 "Capacitors_THT:CP_Axial_L11.0mm_D5.0mm_P18.00mm_Horizontal" H 10088 3600 30  0001 C CNN
 F 3 "" H 10050 3750 60  0000 C CNN
 	1    10050 3750
@@
 	9000 3550 9150 3550
 $Comp
-L Device:LED D?
+L Device:LED D1
 U 1 1 5C81702D
 P 9500 4850
-F 0 "D?" H 9491 5066 50  0000 C CNN
+F 0 "D1" H 9491 5066 50  0000 C CNN
 F 1 "LED" H 9491 4975 50  0000 C CNN
-F 2 "" H 9500 4850 50  0001 C CNN
+F 2 "Capacitors_THT:CP_Axial_L11.0mm_D5.0mm_P18.00mm_Horizontal" H 9500 4850 50  0001 C CNN
 F 3 "~" H 9500 4850 50  0001 C CNN
 	1    9500 4850
@@
 $EndComp
 $Comp
-L Device:LED D?
+L Device:LED D2
 U 1 1 5C81727F
 P 10000 4850
-F 0 "D?" H 9991 5066 50  0000 C CNN
+F 0 "D2" H 9991 5066 50  0000 C CNN
 F 1 "LED" H 9991 4975 50  0000 C CNN
-F 2 "" H 10000 4850 50  0001 C CNN
+F 2 "Capacitors_THT:CP_Axial_L11.0mm_D5.0mm_P18.00mm_Horizontal" H 10000 4850 50  0001 C CNN
 F 3 "~" H 10000 4850 50  0001 C CNN
 	1    10000 4850
@@
 $EndComp
 $Comp
-L Device:Q_NPN_BCE Q?
+L Device:Q_NPN_BCE Q1
 U 1 1 5C8175BD
 P 9450 5400
-F 0 "Q?" H 9641 5446 50  0000 L CNN
+F 0 "Q1" H 9641 5446 50  0000 L CNN
 F 1 "Q_NPN_BCE" H 9641 5355 50  0000 L CNN
-F 2 "" H 9650 5500 50  0001 C CNN
+F 2 "Capacitors_THT:CP_Axial_L11.0mm_D5.0mm_P18.00mm_Horizontal" H 9650 5500 50  0001 C CNN
 F 3 "~" H 9450 5400 50  0001 C CNN
 	1    9450 5400
@@
 $EndComp
 $Comp
-L Device:Q_NPN_BCE Q?
+L Device:Q_NPN_BCE Q2
 U 1 1 5C81765A
 P 9950 5400
-F 0 "Q?" H 10141 5446 50  0000 L CNN
+F 0 "Q2" H 10141 5446 50  0000 L CNN
 F 1 "Q_NPN_BCE" H 10141 5355 50  0000 L CNN
-F 2 "" H 10150 5500 50  0001 C CNN
+F 2 "Sensores_e_componentes_SL:TCRT5000" H 10150 5500 50  0001 C CNN
 F 3 "~" H 9950 5400 50  0001 C CNN
 	1    9950 5400
@@
 $EndComp
 $Comp
-L Device:R R?
+L Device:R R1
 U 1 1 5C817C0F
 P 9500 5100
-F 0 "R?" V 9293 5100 50  0000 C CNN
+F 0 "R1" V 9293 5100 50  0000 C CNN
 F 1 "330" V 9384 5100 50  0000 C CNN
 F 2 "" V 9430 5100 50  0001 C CNN
@@
 $EndComp
 $Comp
-L Device:R R?
+L Device:R R2
 U 1 1 5C817CFF
 P 10000 5100
-F 0 "R?" V 9793 5100 50  0000 C CNN
+F 0 "R2" V 9793 5100 50  0000 C CNN
 F 1 "330" V 9884 5100 50  0000 C CNN
 F 2 "" V 9930 5100 50  0001 C CNN
@@
 	2650 2450 2750 2450
 $Comp
-L Device:LED D?
+L Device:LED D3
 U 1 1 5C81CEED
 P 10500 4850
-F 0 "D?" H 10491 5066 50  0000 C CNN
+F 0 "D3" H 10491 5066 50  0000 C CNN
 F 1 "LED" H 10491 4975 50  0000 C CNN
-F 2 "" H 10500 4850 50  0001 C CNN
+F 2 "Capacitors_THT:CP_Axial_L11.0mm_D5.0mm_P18.00mm_Horizontal" H 10500 4850 50  0001 C CNN
 F 3 "~" H 10500 4850 50  0001 C CNN
 	1    10500 4850
@@
 $EndComp
 $Comp
-L Device:R R?
+L Device:R R7
 U 1 1 5C81CF31
 P 10500 5100
-F 0 "R?" V 10293 5100 50  0000 C CNN
+F 0 "R7" V 10293 5100 50  0000 C CNN
 F 1 "330" V 10384 5100 50  0000 C CNN
 F 2 "" V 10430 5100 50  0001 C CNN
@@
 $EndComp
 $Comp
-L Device:Q_NPN_BCE Q?
+L Device:Q_NPN_BCE Q3
 U 1 1 5C81CFAB
 P 10450 5400
-F 0 "Q?" H 10641 5446 50  0000 L CNN
+F 0 "Q3" H 10641 5446 50  0000 L CNN
 F 1 "Q_NPN_BCE" H 10641 5355 50  0000 L CNN
-F 2 "" H 10650 5500 50  0001 C CNN
+F 2 "Sensores_e_componentes_SL:TCRT5000" H 10650 5500 50  0001 C CNN
 F 3 "~" H 10450 5400 50  0001 C CNN
 	1    10450 5400
@@
 Regulador de tensão +5V
 $Comp
-L Switch:SW_Push SW?
+L Switch:SW_Push SW2
 U 1 1 5C81F63E
 P 8350 5400
-F 0 "SW?" H 8350 5685 50  0000 C CNN
+F 0 "SW2" H 8350 5685 50  0000 C CNN
 F 1 "SW_Push" H 8350 5594 50  0000 C CNN
 F 2 "" H 8350 5600 50  0001 C CNN
@@
 $EndComp
 $Comp
-L Switch:SW_Push SW?
+L Switch:SW_Push SW1
 U 1 1 5C81F7C0
 P 7650 5400
-F 0 "SW?" H 7650 5685 50  0000 C CNN
+F 0 "SW1" H 7650 5685 50  0000 C CNN
 F 1 "SW_Push" H 7650 5594 50  0000 C CNN
 F 2 "" H 7650 5600 50  0001 C CNN

Commit message: Acertada mais questões de libraries
Removi as que nao são necessárias e coloquei os componentes em novas bibliotecas, "Componentes soltos" para a pcb e "Sensores..." para o tcrt e o arduino.
Parts:
- removed C1: 0.33uF, Capacitors_THT:CP_Axial_L11.0mm_D5.0mm_P18.00mm_Horizontal, symbol cyclophone:C
- removed C2: 0.1uF, Capacitors_THT:CP_Axial_L11.0mm_D5.0mm_P18.00mm_Horizontal, symbol cyclophone:C
- removed U1, U2: TCRT5000, symbol Placa_central_v01-rescue:TCRT5000-cyclophone
- added C?: 0,33uF, symbol Device:C
- added C?: 0,1uF, symbol Device:C
- added H?: V8.4 - Lipo, symbol Mechanical:MountingHole_Pad
- added H?: V0 - Lipo, symbol Mechanical:MountingHole_Pad
- added SW?: SW_ON/OFF, symbol Switch:SW_SPST
- added U?: L298P, symbol Driver_Motor:L298P
- added U? (x2): TCRT5000, symbol Sensores_e_componentes_SL:TCRT5000
- SW1: value SW_Push -> SW_comando1
- SW2: value SW_Push -> SW_comando2
Connections:
- wire segments 29 -> 35
Changed lines of the file:
@@
-$EndComp
-$Comp
-L Placa_central_v01-rescue:TCRT5000-cyclophone U2
-U 1 1 5C812FD5
-P 9450 2400
-F 0 "U2" H 9450 2550 60  0000 C CNN
-F 1 "TCRT5000" H 9450 2650 60  0000 C CNN
-F 2 "" H 9450 2400 60  0001 C CNN
-F 3 "" H 9450 2400 60  0000 C CNN
-	1    9450 2400
-	1    0    0    -1
 $EndComp
 $Comp
@@
 	9950 2700 10000 2700
 $Comp
-L Placa_central_v01-rescue:TCRT5000-cyclophone U1
-U 1 1 5C8139FF
-P 9450 1450
-F 0 "U1" H 9450 1600 60  0000 C CNN
-F 1 "TCRT5000" H 9450 1700 60  0000 C CNN
-F 2 "" H 9450 1450 60  0001 C CNN
-F 3 "" H 9450 1450 60  0000 C CNN
-	1    9450 1450
-	1    0    0    -1
-$EndComp
-$Comp
 L Device:R R3
 U 1 1 5C813A06
@@
 Wire Wire Line
 	9950 1950 10050 1950
-Connection ~ 9950 1750
 Wire Wire Line
 	9950 2700 9950 2900
 Wire Wire Line
 	9950 2900 10050 2900
-Connection ~ 9950 2700
 Text GLabel 8850 2450 0    50   Input ~ 0
 5V
@@
 Text GLabel 10050 2900 2    50   Input ~ 0
 Encoder2
-$Comp
-L Regulator_Linear:L7805 U3
-U 1 1 5C81568D
-P 9600 3550
-F 0 "U3" H 9600 3792 50  0000 C CNN
-F 1 "L7805" H 9600 3701 50  0000 C CNN
-F 2 "" H 9625 3400 50  0001 L CIN
-F 3 "http://www.st.com/content/ccc/resource/technical/document/datasheet/41/4f/b3/b0/12/d4/47/88/CD00000444.pdf/files/CD00000444.pdf/jcr:content/translations/en.CD00000444.pdf" H 9600 3500 50  0001 C CNN
-	1    9600 3550
-	1    0    0    -1
-$EndComp
 Text GLabel 10250 3950 2    50   Input ~ 0
 GND
-$Comp
-L cyclophone:C C1
-U 1 1 5C81583B
-P 9150 3750
-F 0 "C1" H 9265 3788 40  0000 L CNN
-F 1 "0.33uF" H 9265 3712 40  0000 L CNN
-F 2 "Capacitors_THT:CP_Axial_L11.0mm_D5.0mm_P18.00mm_Horizontal" H 9188 3600 30  0001 C CNN
-F 3 "" H 9150 3750 60  0000 C CNN
-	1    9150 3750
-	1    0    0    -1
-$EndComp
-$Comp
-L cyclophone:C C2
-U 1 1 5C8158B3
-P 10050 3750
-F 0 "C2" H 10165 3788 40  0000 L CNN
-F 1 "0.1uF" H 10165 3712 40  0000 L CNN
-F 2 "Capacitors_THT:CP_Axial_L11.0mm_D5.0mm_P18.00mm_Horizontal" H 10088 3600 30  0001 C CNN
-F 3 "" H 10050 3750 60  0000 C CNN
-	1    10050 3750
-	1    0    0    -1
-$EndComp
-Wire Wire Line
-	10250 3950 10050 3950
-Connection ~ 10050 3950
-Wire Wire Line
-	10050 3950 9150 3950
-Wire Wire Line
-	9300 3550 9150 3550
-Connection ~ 9150 3550
-Wire Wire Line
-	9900 3550 10050 3550
-Connection ~ 10050 3550
-Wire Wire Line
-	10050 3550 10250 3550
 Text GLabel 10250 3550 2    50   Input ~ 0
 5V
 Text GLabel 9000 3550 0    50   Input ~ 0
 8.4V
-Wire Wire Line
-	9000 3550 9150 3550
 $Comp
 L Device:LED D1
@@
 P 8350 5400
 F 0 "SW2" H 8350 5685 50  0000 C CNN
-F 1 "SW_Push" H 8350 5594 50  0000 C CNN
+F 1 "SW_comando2" H 8350 5594 50  0000 C CNN
 F 2 "" H 8350 5600 50  0001 C CNN
 F 3 "" H 8350 5600 50  0001 C CNN
@@
 P 7650 5400
 F 0 "SW1" H 7650 5685 50  0000 C CNN
-F 1 "SW_Push" H 7650 5594 50  0000 C CNN
+F 1 "SW_comando1" H 7650 5594 50  0000 C CNN
 F 2 "" H 7650 5600 50  0001 C CNN
 F 3 "" H 7650 5600 50  0001 C CNN
@@
 Text GLabel 3900 2750 2    50   Input ~ 0
 Botao1
+$Comp
+L Switch:SW_SPST SW?
+U 1 1 5D0BCA30
+P 6000 5400
+F 0 "SW?" H 6000 5635 50  0000 C CNN
+F 1 "SW_ON/OFF" H 6000 5544 50  0000 C CNN
+F 2 "" H 6000 5400 50  0001 C CNN
+F 3 "" H 6000 5400 50  0001 C CNN
+	1    6000 5400
+	1    0    0    -1
+$EndComp
+$Comp
+L Mechanical:MountingHole_Pad H?
+U 1 1 5D0BE091
+P 3650 5450
+F 0 "H?" H 3750 5501 50  0000 L CNN
+F 1 "V8.4 - Lipo" H 3750 5410 50  0000 L CNN
+F 2 "" H 3650 5450 50  0001 C CNN
+F 3 "~" H 3650 5450 50  0001 C CNN
+	1    3650 5450
+	1    0    0    -1
+$EndComp
+$Comp
+L Mechanical:MountingHole_Pad H?
+U 1 1 5D0BE14B
+P 3850 5750
+F 0 "H?" H 3950 5801 50  0000 L CNN
+F 1 "V0 - Lipo" H 3950 5710 50  0000 L CNN
+F 2 "" H 3850 5750 50  0001 C CNN
+F 3 "~" H 3850 5750 50  0001 C CNN
+	1    3850 5750
+	1    0    0    -1
+$EndComp
+$Comp
+L Driver_Motor:L298P U?
+U 1 1 5D0BE849
+P 5650 2850
+F 0 "U?" H 5650 3728 50  0000 C CNN
+F 1 "L298P" H 5650 3637 50  0000 C CNN
+F 2 "" H 5800 3100 50  0001 C CNN
+F 3 "http://www.st.com/st-web-ui/static/active/en/resource/technical/document/datasheet/CD00000240.pdf" H 5800 3100 50  0001 C CNN
+	1    5650 2850
+	1    0    0    -1
+$EndComp
+$Comp
+L Device:C C?
+U 1 1 5D0BC666
+P 9150 3750
+F 0 "C?" H 9265 3796 50  0000 L CNN
+F 1 "0,33uF" H 9265 3705 50  0000 L CNN
+F 2 "" H 9188 3600 50  0001 C CNN
+F 3 "~" H 9150 3750 50  0001 C CNN
+	1    9150 3750
+	1    0    0    -1
+$EndComp
+$Comp
+L Regulator_Linear:L7805 U3
+U 1 1 5C81568D
+P 9600 3550
+F 0 "U3" H 9600 3792 50  0000 C CNN
+F 1 "L7805" H 9600 3701 50  0000 C CNN
+F 2 "" H 9625 3400 50  0001 L CIN
+F 3 "http://www.st.com/content/ccc/resource/technical/document/datasheet/41/4f/b3/b0/12/d4/47/88/CD00000444.pdf/files/CD00000444.pdf/jcr:content/translations/en.CD00000444.pdf" H 9600 3500 50  0001 C CNN
+	1    9600 3550
+	1    0    0    -1
+$EndComp
+Wire Wire Line
+	9000 3550 9150 3550
+Wire Wire Line
+	9150 3900 9150 3950
+Wire Wire Line
+	9150 3600 9150 3550
+Connection ~ 9150 3550
+Wire Wire Line
+	9150 3550 9300 3550
+$Comp
+L Device:C C?
+U 1 1 5D0BDB83
+P 10050 3750
+F 0 "C?" H 10165 3796 50  0000 L CNN
+F 1 "0,1uF" H 10165 3705 50  0000 L CNN
+F 2 "" H 10088 3600 50  0001 C CNN
+F 3 "~" H 10050 3750 50  0001 C CNN
+	1    10050 3750
+	1    0    0    -1
+$EndComp
+Wire Wire Line
+	9900 3550 10050 3550
+Wire Wire Line
+	9150 3950 9600 3950
+Wire Wire Line
+	10050 3600 10050 3550
+Connection ~ 10050 3550
+Wire Wire Line
+	10050 3550 10250 3550
+Wire Wire Line
+	10050 3900 10050 3950
+Connection ~ 10050 3950
+Wire Wire Line
+	10050 3950 10250 3950
+Wire Wire Line
+	9600 3850 9600 3950
+Connection ~ 9600 3950
+Wire Wire Line
+	9600 3950 10050 3950
+$Comp
+L Sensores_e_componentes_SL:TCRT5000 U?
+U 1 1 5D0BF882
+P 9450 1450
+F 0 "U?" H 9450 1937 60  0000 C CNN
+F 1 "TCRT5000" H 9450 1831 60  0000 C CNN
+F 2 "" H 9450 1450 60  0000 C CNN
+F 3 "" H 9450 1450 60  0000 C CNN
+	1    9450 1450
+	1    0    0    -1
+$EndComp
+Connection ~ 9950 1750
+$Comp
+L Sensores_e_componentes_SL:TCRT5000 U?
+U 1 1 5D0BF8FC
+P 9450 2400
+F 0 "U?" H 9450 2887 60  0000 C CNN
+F 1 "TCRT5000" H 9450 2781 60  0000 C CNN
+F 2 "" H 9450 2400 60  0000 C CNN
+F 3 "" H 9450 2400 60  0000 C CNN
+	1    9450 2400
+	1    0    0    -1
+$EndComp
+Connection ~ 9950 2700
 $EndSCHEMATC

Commit message: Organizado Pcb
Adicionado circuito de alimentação
Parts:
- removed C?: 0,33uF, symbol Device:C
- removed C?: 0,1uF, symbol Device:C
- removed D2, D3: LED, Capacitors_THT:CP_Axial_L11.0mm_D5.0mm_P18.00mm_Horizontal, symbol Device:LED
- removed Q1: Q_NPN_BCE, Capacitors_THT:CP_Axial_L11.0mm_D5.0mm_P18.00mm_Horizontal, symbol Device:Q_NPN_BCE
- removed Q2, Q3: Q_NPN_BCE, Sensores_e_componentes_SL:TCRT5000, symbol Device:Q_NPN_BCE
- removed R2, R7: 330, symbol Device:R
- removed SW2: SW_comando2, symbol Switch:SW_Push
- removed U3: L7805, symbol Regulator_Linear:L7805
- removed U?: L298P, symbol Driver_Motor:L298P
- added D?: DiodoProtecao-4A, symbol Device:D
- added D?: LedVerde, Capacitors_THT:CP_Axial_L11.0mm_D5.0mm_P18.00mm_Horizontal, symbol Device:LED
- added F?: Fuse-4A, symbol Device:Fuse
- added H?: FurosPonteH, symbol Mechanical:MountingHole
- added J?: PinoChargeBateriaV++, symbol Connector:Conn_01x01_Female
- added J?: PinoChargeBateriaGND, symbol Connector:Conn_01x01_Female
- added J?: Conn_01x02_Motor1, symbol Connector:Conn_01x02_Female
- added J?: Conn_01x02_Motor2, symbol Connector:Conn_01x02_Female
- added J?: Conn_01x01_Motor1PWM, symbol Connector:Conn_01x01_Female
- added J?: Conn_01x01_Motor1Dir1, symbol Connector:Conn_01x01_Female
- added J?: Conn_01x01_Motor1Dir2, symbol Connector:Conn_01x01_Female
- added J?: Conn_01x01_Motor2Dir1, symbol Connector:Conn_01x01_Female
- added J?: Conn_01x01_Motor2Dir2, symbol Connector:Conn_01x01_Female
- added J?: Conn_01x01_Motor2PWM, symbol Connector:Conn_01x01_Female
- added J?: Conn_01x01_8.4VPonteH, symbol Connector:Conn_01x01_Female
- added J?: Conn_01x01_GNDPonteH, symbol Connector:Conn_01x01_Female
- added J?: Conn_01x01_5VPonteH, symbol Connector:Conn_01x01_Female
- added J?: Conn_01x01_5VPlacaSensores, symbol Connector:Conn_01x01_Female
- added J?: Conn_01x01_GNDPlacaSensores, symbol Connector:Conn_01x01_Female
- added R?: 330, symbol Device:R
- added RPullDown: R, symbol Device:R
- added SW?: SW_AlimentacaoPlacaSensores, symbol Switch:SW_DPDT_x2
- D1: value LED -> LedAzul
- H?: value V0 - Lipo -> GND - Lipo
Connections:
- net labels added: 5VArduino, 5VPonteH, Botao2, LedAzul, Motor11, Motor12, Motor1Dir1, Motor1Dir2, Motor1PWM, Motor21, Motor22, Motor2Dir1, Motor2Dir2, Motor2PWM, VccSensores
- wire segments 35 -> 86
- no-connect marks 3 -> 5
Other:
- note added: "Arduino Nano V3.x"
- note added: "Botoes da pcb"
- note added: "Circuito de Alimentação da placa e Sistema de proteção"
- note added: "Leds da pcb"
- note added: "Ponte H - Pinos soltos"
- note added: "Switch de alimentação da placa de sensores"
- note removed: "Regulador de tensão +5V"
- moved on the sheet: A1, D1, H?, R1, SW1, SW?
