File: Placa central/Placa_central_v01/Placa_central_v01.kicad_pcb (KiCad board)
At the start: 0 parts

Commit message: Adicionados os componentes à PBC - ainda não posicionados corretamente
Parts:
- added A1: Arduino_Nano_v3.x, Sensores_e_componentes_SL:Arduino_Nano, F.Cu at (118.4, 84.8)
- added D1: DiodoProtecao-5A, Diode_THT:D_DO-27_P15.24mm_Horizontal, F.Cu at (601.5, 94.5)
- added D2: DiodoZener6.8V, Diode_THT:D_DO-35_SOD27_P10.16mm_Horizontal, F.Cu at (111.3, 260.1)
- added D3: LedBateriaVermelho, LED_THT:LED_D3.0mm, F.Cu at (53.3, 203.2)
- added D4: LedAzul, LED_THT:LED_D3.0mm, F.Cu at (390.7, 229.6)
- added D5: LedVerde, LED_THT:LED_D3.0mm, F.Cu at (381.5, 216.9)
- added F1: Fuse-5A, Fuse:Fuseholder_Cylinder-5x20mm_Stelvio-Kontek_PTF78_Horizontal_Open, F.Cu at (623.8, 123.4)
- added F2: Fuse-3A, Fuse:Fuseholder_Cylinder-5x20mm_Stelvio-Kontek_PTF78_Horizontal_Open, F.Cu at (33.0, 41.7)
- added F3: Fuse-3A, Fuse:Fuseholder_Cylinder-5x20mm_Stelvio-Kontek_PTF78_Horizontal_Open, F.Cu at (413.5, -17.8)
- added H1: V8.4 - Lipo, Connector_Wire:SolderWirePad_1x01_Drill1.5mm, F.Cu at (625.9, 96.0)
- added H2: GND - Lipo, Connector_Wire:SolderWirePad_1x01_Drill1.5mm, F.Cu at (649.2, 223.0)
- added H3: FuroBateria, Sensores_e_componentes_SL:Bateria, F.Cu at (113.3, 43.2)
- added H4: FurosPonteH, Sensores_e_componentes_SL:Ponte_H_furos, F.Cu at (69.1, 92.5)
- added J1: PinoCheckBateriaVcc, Connector_PinSocket_2.54mm:PinSocket_1x01_P2.54mm_Vertical, F.Cu at (611.1, 165.1)
- added J10: Conn_01x01_Arduino11, Connector_PinSocket_2.54mm:PinSocket_1x01_P2.54mm_Vertical, F.Cu at (174.2, 87.9)
- added J11: Conn_01x01_Arduino12, Connector_PinSocket_2.54mm:PinSocket_1x01_P2.54mm_Vertical, F.Cu at (178.8, 89.9)
- added J12: Conn_01x01_Arduino13, Connector_PinSocket_2.54mm:PinSocket_1x01_P2.54mm_Vertical, F.Cu at (173.7, 93.0)
- added J13: Conn_01x01_Arduino14, Connector_PinSocket_2.54mm:PinSocket_1x01_P2.54mm_Vertical, F.Cu at (76.2, 139.7)
- added J14: Conn_01x01_Arduino15, Connector_PinSocket_2.54mm:PinSocket_1x01_P2.54mm_Vertical, F.Cu at (188.2, 0.29)
- added J15: Conn_01x01_Arduino16, Connector_PinSocket_2.54mm:PinSocket_1x01_P2.54mm_Vertical, F.Cu at (142.6, 45.3)
- added J16: Conn_01x01_Motor1PonteHPCB, Connector_Wire:SolderWirePad_1x01_Drill1.5mm, F.Cu at (33.5, 49.8)
- added J17: PinoChargeBateriaGND, Connector_Wire:SolderWirePad_1x01_Drill1.5mm, F.Cu at (649.7, 207.3)
- added J18: Conn_01x01_Arduino19, Connector_PinSocket_2.54mm:PinSocket_1x01_P2.54mm_Vertical, F.Cu at (171.5, 15.3)
- added J19: Conn_01x01_Arduino20, Connector_PinSocket_2.54mm:PinSocket_1x01_P2.54mm_Vertical, F.Cu at (177.7, 8.79)
- added J2: Conn_01x02_ArduinoTxRx, Connector_PinSocket_2.54mm:PinSocket_1x02_P2.54mm_Vertical, F.Cu at (184.4, 57.4)
- added J20: Conn_01x01_Arduino21, Connector_PinSocket_2.54mm:PinSocket_1x01_P2.54mm_Vertical, F.Cu at (183.6, 3.24)
- added J21: Conn_01x01_Arduino22, Connector_PinSocket_2.54mm:PinSocket_1x01_P2.54mm_Vertical, F.Cu at (239.3, 106.2)
- added J22: Conn_01x01_Arduino23, Connector_PinSocket_2.54mm:PinSocket_1x01_P2.54mm_Vertical, F.Cu at (231.6, 79.8)
- added J23: Conn_01x01_Arduino24, Connector_PinSocket_2.54mm:PinSocket_1x01_P2.54mm_Vertical, F.Cu at (142.6, 49.9)
- added J24: Conn_01x01_Arduino25, Connector_PinSocket_2.54mm:PinSocket_1x01_P2.54mm_Vertical, F.Cu at (163.8, 30.1)
- added J25: Conn_01x01_Arduino26, Connector_PinSocket_2.54mm:PinSocket_1x01_P2.54mm_Vertical, F.Cu at (168.4, 25.5)
- added J26: Conn_02x08_Odd_Even, Connector_IDC:IDC-Header_2x08_P2.54mm_Horizontal, F.Cu at (106.2, 137.2)
- added J27: Conn_01x01_Motor2PonteHPCB, Connector_Wire:SolderWirePad_1x01_Drill1.5mm, F.Cu at (395.7, -15.7)
- added J28: Conn_01x01_Motor1PCBMotor, Connector_Wire:SolderWirePad_1x01_Drill1.5mm, F.Cu at (33.0, 12.2)
- added J29: Conn_01x01_Motor2PCBMotor, Connector_Wire:SolderWirePad_1x01_Drill1.5mm, F.Cu at (457.7, -16.3)
- added J3: Conn_01x01_ArduinoReset, Connector_PinSocket_2.54mm:PinSocket_1x01_P2.54mm_Vertical, F.Cu at (179.3, 64.0)
- added J37: Conn_01x01_8.4VPonteH, Connector_Wire:SolderWirePad_1x01_Drill1.2mm, F.Cu at (150.2, 27.8)
- added J38: Conn_01x01_5VPonteH, Connector_Wire:SolderWirePad_1x01_Drill1.2mm, F.Cu at (158.2, 33.9)
- added J39: Conn_01x01_GNDPonteH, Connector_Wire:SolderWirePad_1x01_Drill1.2mm, F.Cu at (158.3, 21.2)
- added J4: Conn_01x01_Arduino5, Connector_PinSocket_2.54mm:PinSocket_1x01_P2.54mm_Vertical, F.Cu at (179.3, 69.6)
- added J40: Conn_01x01_Motor1PWM, Connector_Wire:SolderWirePad_1x01_Drill0.8mm, F.Cu at (146.9, 49.6)
- added J41: Conn_01x01_Motor1Dir1, Connector_Wire:SolderWirePad_1x01_Drill0.8mm, F.Cu at (165.1, 77.7)
- added J42: Conn_01x01_Motor1Dir2, Connector_Wire:SolderWirePad_1x01_Drill0.8mm, F.Cu at (168.1, 29.8)
- added J43: Conn_01x01_Motor2Dir1, Connector_Wire:SolderWirePad_1x01_Drill0.8mm, F.Cu at (163.0, 34.4)
- added J44: Conn_01x01_Motor2Dir2, Connector_Wire:SolderWirePad_1x01_Drill0.8mm, F.Cu at (172.7, 22.3)
- added J45: Conn_01x01_Motor2PWM, Connector_Wire:SolderWirePad_1x01_Drill0.8mm, F.Cu at (186.6, 12.1)
- added J48: Conn_01x01_5VEncoderEsq, Connector_Wire:SolderWirePad_1x01_Drill0.8mm, F.Cu at (180.4, 17.7)
- added J49: Conn_01x01_OutputEncoderEsq, Connector_PinSocket_2.54mm:PinSocket_1x01_P2.54mm_Vertical, F.Cu at (186.9, 7.84)
- added J5: Conn_01x01_Arduino6, Connector_PinSocket_2.54mm:PinSocket_1x01_P2.54mm_Vertical, F.Cu at (178.8, 73.7)
- added J50: Conn_01x01_GNDEncoderEsq, Connector_Wire:SolderWirePad_1x01_Drill0.8mm, F.Cu at (104.3, 233.0)
- added J51: Conn_01x01_5VEncoderDir, Connector_Wire:SolderWirePad_1x01_Drill0.8mm, F.Cu at (219.5, 69.6)
- added J52: Conn_01x01_OutputEncoderDir, Connector_PinSocket_2.54mm:PinSocket_1x01_P2.54mm_Vertical, F.Cu at (147.2, 45.3)
- added J53: Conn_01x01_GNDEncoderDir, Connector_Wire:SolderWirePad_1x01_Drill0.8mm, F.Cu at (108.4, 233.0)
- added J6: Conn_01x01_Arduino7, Connector_PinSocket_2.54mm:PinSocket_1x01_P2.54mm_Vertical, F.Cu at (178.8, 77.7)
- added J7: Conn_01x01_Arduino8, Connector_PinSocket_2.54mm:PinSocket_1x01_P2.54mm_Vertical, F.Cu at (174.2, 80.3)
- added J8: Conn_01x01_Arduino9, Connector_PinSocket_2.54mm:PinSocket_1x01_P2.54mm_Vertical, F.Cu at (220.5, 97.5)
- added J9: Conn_01x01_Arduino10, Connector_PinSocket_2.54mm:PinSocket_1x01_P2.54mm_Vertical, F.Cu at (178.8, 84.8)
- added Q1: BC548, Package_TO_SOT_THT:TO-92_Wide, F.Cu at (27.9, 180.8)
- added Q2: BC548, Package_TO_SOT_THT:TO-92_Wide, F.Cu at (31.5, 197.6)
- added R1: RBatCheck10K, Resistor_THT:R_Axial_DIN0207_L6.3mm_D2.5mm_P10.16mm_Horizontal, F.Cu at (601.0, 154.4)
- added R2: R6K6MedidorDeBateria, Resistor_THT:R_Axial_DIN0207_L6.3mm_D2.5mm_P10.16mm_Horizontal, F.Cu at (138.2, 239.8)
- added R3: R1KMedidorDeBateria, Resistor_THT:R_Axial_DIN0207_L6.3mm_D2.5mm_P10.16mm_Horizontal, F.Cu at (28.4, 158.5)
- added R4: R10KMedidorDeBateria, Resistor_THT:R_Axial_DIN0207_L6.3mm_D2.5mm_P10.16mm_Horizontal, F.Cu at (86.4, 290.1)
- added R5: RMedidorDeBateria1K, Resistor_THT:R_Axial_DIN0207_L6.3mm_D2.5mm_P10.16mm_Horizontal, F.Cu at (50.3, 185.4)
- added R6: R330LedAzul, Resistor_THT:R_Axial_DIN0207_L6.3mm_D2.5mm_P10.16mm_Horizontal, F.Cu at (357.1, 206.8)
- added R7: R330LedVerde, Resistor_THT:R_Axial_DIN0207_L6.3mm_D2.5mm_P10.16mm_Horizontal, F.Cu at (378.5, 206.8)
- added RPullDown1: R10KPullDown, Resistor_THT:R_Axial_DIN0207_L6.3mm_D2.5mm_P10.16mm_Horizontal, F.Cu at (255.5, -73.2)
- added SW1: SW_ON/OFF, Sensores_e_componentes_SL:BotaoOnOff, F.Cu at (602.5, 74.2)
- added SW3: SW_comando1, Button_Switch_THT:SW_PUSH_6mm_H5mm, F.Cu at (238.3, -56.4)
Other:
- copper layers 0 -> 2
- net class Default added: clearance 0.2, trace_width 0.25, via_dia 0.8, via_drill 0.4
