File: Placa sensores/Placa_sensores v1_2/Placa_sensores_v1_2.sch (KiCad schematic (older format))
At the start: 37 parts, among them J1 Conn_01x01_Female, J10 Conn_01x01_Female, J11 Conn_01x01_Female, J12 Conn_01x01_Female, J2 Conn_01x01_Female, J3 Conn_01x01_Female, J4 Conn_01x01_Female, J5 Conn_01x01_Female, J6 Conn_01x01_Female, J7 Conn_01x01_Female, J8 Conn_01x01_Female, J9 Conn_01x01_Female, U1 TCRT5000, U2 TCRT5000, U3 TCRT5000, U4 TCRT5000, U5 TCRT5000, U6 TCRT5000, U7 TCRT5000, U8 TCRT5000, U9 TCRT5000

Commit message: Acertado a placa de sensores
Acertado biblioteca, esquemático, conexão entre as placas e só.
Parts:
- removed J1, J10, J11, J12, J2, J3, J4, J5, J6, J7, J8, J9: Conn_01x01_Female, Connector_PinSocket_2.54mm:PinSocket_1x01_P2.54mm_Vertical, symbol Connector:Conn_01x01_Female
- removed U1, U2, U3, U4, U5, U6, U7, U8, U9: TCRT5000, Tcrt5000_e_afins:TCRT50002, symbol Tcrt5000_e_afins:TCRT5000
- added D2, D3, D4, D5, D6, D7, D8, D9: LED, LED_THT:LED_D3.0mm, symbol Device:LED
- added J1: Conn_02x08_Odd_Even, Connector_IDC:IDC-Header_2x08_P2.54mm_Horizontal, symbol Connector_Generic:Conn_02x08_Odd_Even
- added Q1, Q2, Q3, Q4, Q5, Q6, Q7, Q8, Q9: 2n2222a, Package_TO_SOT_THT:TO-92_Wide, symbol Transistor_BJT:BC338
- added R16, R29, R30, R31, R32, R36: R4k7Divisor, Resistor_THT:R_Axial_DIN0207_L6.3mm_D2.5mm_P10.16mm_Horizontal, symbol Device:R
- added R17, R18, R19, R20, R33: R330Emissor, Resistor_THT:R_Axial_DIN0207_L6.3mm_D2.5mm_P10.16mm_Horizontal, symbol Device:R
- added R21, R22, R23, R24, R34: R2kLed, Resistor_THT:R_Axial_DIN0207_L6.3mm_D2.5mm_P10.16mm_Horizontal, symbol Device:R
- added R25, R26, R27, R28, R35: R1M2Transsistor, Resistor_THT:R_Axial_DIN0207_L6.3mm_D2.5mm_P10.16mm_Horizontal, symbol Device:R
- added U1, U2, U3, U4, U5, U6, U7, U8, U9: TCRT5000, Sensores_SL:TCRT5000Extendido, symbol Sensores_SL:TCRT5000
- D1: value LED - ON/OFF -> LED
- R1: value 330 -> R4k7Divisor
- R10, R9: value 330 -> R2kLed
- R11, R2: value 330 -> R1M2Transsistor
- R12, R13: value 10k -> R1M2Transsistor
- R14, R15: value 10k -> R4k7Divisor
- R3: value 330 -> R330Emissor
- R4, R8: value 10k -> R2kLed
- R5, R6, R7: value 10k -> R330Emissor
Connections:
- net labels added: 5V, Gnd, Sensor1, Sensor2, Sensor3, Sensor4, Sensor5, Sensor6, Sensor7
- net labels removed: S1, S2, S3, S4, S5, S6, S7, VCC
- wire segments 143 -> 200
- no-connect marks 0 -> 5
Other:
- note added: "Circuitos dos Sensores"
- note added: "Pinos de conexão"
- note added: "Sensor 1"
- note added: "Sensor 2"
- note added: "Sensor 3"
- note added: "Sensor 4"
- note added: "Sensor 5"
- note added: "Sensor 6"
- note added: "Sensor 7"
- note added: "Sensor Direita"
- note added: "Sensor Esquerda"
- note removed: "Conectores dos sensores"
- note removed: "Led para indicar alimentação da placa"
- note removed: "Modulos Tcrt5000\n"
- note removed: "Pad livre para referência de multímetro\n"
